File: pcb/mini-talkie.kicad_pcb (KiCad board)
At the start: 2 copper layers, 0 parts

Commit message: schematic almost done
Parts:
- added C1: 2.2u, Capacitor_SMD:C_0603_1608Metric_Pad1.08x0.95mm_HandSolder, F.Cu at (128.7, 78.3)
- added C10: 10u, Capacitor_SMD:C_0805_2012Metric_Pad1.18x1.45mm_HandSolder, F.Cu at (128.9, 101.6)
- added C11: 10u, Capacitor_SMD:C_0805_2012Metric_Pad1.18x1.45mm_HandSolder, F.Cu at (128.9, 104.6)
- added C12: 10u, Capacitor_SMD:C_0805_2012Metric_Pad1.18x1.45mm_HandSolder, F.Cu at (128.9, 107.6)
- added C13: 10u, Capacitor_SMD:C_0805_2012Metric_Pad1.18x1.45mm_HandSolder, F.Cu at (128.9, 110.6)
- added C14: 100n, Capacitor_SMD:C_0603_1608Metric_Pad1.08x0.95mm_HandSolder, F.Cu at (133.0, 78.3)
- added C15: 1u, Capacitor_SMD:C_0603_1608Metric_Pad1.08x0.95mm_HandSolder, F.Cu at (133.0, 80.8)
- added C16: 1u, Capacitor_SMD:C_0603_1608Metric_Pad1.08x0.95mm_HandSolder, F.Cu at (133.0, 83.3)
- added C17: 10u, Capacitor_SMD:C_0603_1608Metric_Pad1.08x0.95mm_HandSolder, F.Cu at (133.0, 85.8)
- added C18: 100n, Capacitor_SMD:C_0603_1608Metric_Pad1.08x0.95mm_HandSolder, F.Cu at (133.0, 88.3)
- added C19: 100n, Capacitor_SMD:C_0603_1608Metric_Pad1.08x0.95mm_HandSolder, F.Cu at (133.0, 90.8)
- added C2: 2.2u, Capacitor_SMD:C_0603_1608Metric_Pad1.08x0.95mm_HandSolder, F.Cu at (128.7, 80.8)
- added C20: 10u, Capacitor_SMD:C_0805_2012Metric_Pad1.18x1.45mm_HandSolder, F.Cu at (128.9, 113.6)
- added C3: 100n, Capacitor_SMD:C_0603_1608Metric_Pad1.08x0.95mm_HandSolder, F.Cu at (128.7, 83.3)
- added C4: 100n, Capacitor_SMD:C_0603_1608Metric_Pad1.08x0.95mm_HandSolder, F.Cu at (128.7, 85.8)
- added C5: 100n, Capacitor_SMD:C_0603_1608Metric_Pad1.08x0.95mm_HandSolder, F.Cu at (128.7, 88.3)
- added C6: 100n, Capacitor_SMD:C_0603_1608Metric_Pad1.08x0.95mm_HandSolder, F.Cu at (128.7, 90.8)
- added C7: 100n, Capacitor_SMD:C_0603_1608Metric_Pad1.08x0.95mm_HandSolder, F.Cu at (128.7, 93.3)
- added C8: 10u, Capacitor_SMD:C_0805_2012Metric_Pad1.18x1.45mm_HandSolder, F.Cu at (128.9, 98.6)
- added C9: 100n, Capacitor_SMD:C_0603_1608Metric_Pad1.08x0.95mm_HandSolder, F.Cu at (128.7, 95.8)
- added D1: PMEG3020EH, Diode_SMD:D_SMA_Handsoldering, F.Cu at (144.6, 123.3)
- added D2: ORANGE, LED_SMD:LED_0805_2012Metric_Pad1.15x1.40mm_HandSolder, F.Cu at (168.0, 91.3)
- added FB1: 600@100, Inductor_SMD:L_0603_1608Metric_Pad1.05x0.95mm_HandSolder, F.Cu at (133.0, 93.3)
- added J1: SWD, Connector_JST:JST_SH_BM03B-SRSS-TB_1x03-1MP_P1.00mm_Vertical, F.Cu at (135.2, 100.2)
- added J2: USB_C_Receptacle_USB2.0_16P, Connector_USB:USB_C_Receptacle_GCT_USB4085, F.Cu at (129.3, 116.7)
- added J3: BATT, Connector_JST:JST_PH_S2B-PH-K_1x02_P2.00mm_Horizontal, F.Cu at (156.3, 97.0)
- added J4: SPEAKER, Connector_JST:JST_PH_S2B-PH-K_1x02_P2.00mm_Horizontal, F.Cu at (164.3, 97.0)
- added MK1: Microphone, Mini_Talkie:PUI_THT-2, F.Cu at (146.4, 77.8)
- added Q1: AO3401A, Package_TO_SOT_SMD:SOT-23, F.Cu at (163.2, 92.0)
- added R1: 10k, Resistor_SMD:R_0603_1608Metric_Pad0.98x0.95mm_HandSolder, F.Cu at (133.0, 95.8)
- added R2: 5.1k, Resistor_SMD:R_0603_1608Metric_Pad0.98x0.95mm_HandSolder, F.Cu at (137.4, 78.3)
- added R3: 5.1k, Resistor_SMD:R_0603_1608Metric_Pad0.98x0.95mm_HandSolder, F.Cu at (137.4, 80.8)
- added R4: 10k, Resistor_SMD:R_0603_1608Metric_Pad0.98x0.95mm_HandSolder, F.Cu at (137.4, 83.3)
- added R5: 10k, Resistor_SMD:R_0603_1608Metric_Pad0.98x0.95mm_HandSolder, F.Cu at (137.4, 85.8)
- added R6: 10k, Resistor_SMD:R_0603_1608Metric_Pad0.98x0.95mm_HandSolder, F.Cu at (137.4, 88.3)
- added R7: 5.1k, Resistor_SMD:R_0603_1608Metric_Pad0.98x0.95mm_HandSolder, F.Cu at (137.4, 90.8)
- added R8: 1k, Resistor_SMD:R_0805_2012Metric_Pad1.20x1.40mm_HandSolder, F.Cu at (168.2, 105.7)
- added SW1: SW_SP3T, Mini_Talkie:CK_SW_SP3T_OS103011MA7QP1C, F.Cu at (161.3, 77.8)
- added SW2: SW_SPDT, Button_Switch_THT:SW_Slide_SPDT_Angled_CK_OS102011MA1Q, F.Cu at (157.6, 107.5)
- added SW3: SW_SPST, Button_Switch_THT:SW_SPST_Omron_B3F-315x_Angled, F.Cu at (142.8, 116.3)
- added TP1: ~{RST}, TestPoint:TestPoint_Pad_D2.0mm, F.Cu at (133.3, 105.4)
- added TP2: BOOT0, TestPoint:TestPoint_Pad_D2.0mm, F.Cu at (133.3, 109.4)
- added U1: STM32H503CBTx, Package_QFP:LQFP-48_7x7mm_P0.5mm, F.Cu at (159.0, 120.4)
- added U2: Wio-SX1262, Mini_Talkie:Seeed_SMD-12, F.Cu at (147.0, 102.0)
- added U3: PAM8302AAS, Package_SO:MSOP-8_3x3mm_P0.65mm, F.Cu at (157.0, 92.1)
- added U4: MCP73831-2-OT, Package_TO_SOT_SMD:SOT-23-5, F.Cu at (167.3, 117.1)
- added U5: RT9080, Package_TO_SOT_SMD:TSOT-23-5, F.Cu at (167.3, 121.7)

Commit message: get started with layout
Parts:
- moved R2 66.0 mm to (155.4, 141.8)
- moved R3 56.2 mm to (147.2, 136.1), turned to 90 degrees
- moved R5 50.6 mm to (149.5, 134.9), turned to 90 degrees
- moved SW3 42.5 mm to (165.8, 80.5), turned to -90 degrees
- moved Q1 39.5 mm to (161.1, 131.4), turned to 90 degrees
- moved SW2 36.5 mm to (131.2, 82.2), turned to -90 degrees
- moved C16 33.1 mm to (100.3, 78.4)
- moved C6 33.1 mm to (96.0, 85.9)
- moved C9 33.1 mm to (96.0, 91.0)
- moved R1 33.1 mm to (100.3, 91.0)
- moved C1 33.1 mm to (96.0, 73.4)
- moved C14 33.1 mm to (100.3, 73.4)
- moved C15 33.1 mm to (100.3, 75.9)
- moved C17 33.1 mm to (100.3, 80.9)
- moved C2 33.1 mm to (96.0, 75.9)
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Connections:
- SW1 pad 1: unconnected-(SW1-Pad1) -> /MODE_VA
- SW1 pad 2: unconnected-(SW1-Pad2) -> /MODE_PTT
- SW1 pad 3: unconnected-(SW1-Pad3) -> /MODE_C
- SW1 pad 4: unconnected-(SW1-Pad4) -> /MODE_M
- SW3 pad 1: unconnected-(SW3-A-Pad1) -> /PTT_IN
- SW3 pad 2: unconnected-(SW3-B-Pad2) -> /PTT_OUT
- U1 pad 25: unconnected-(U1-PB12-Pad25) -> /MODE_C
- U1 pad 26: unconnected-(U1-PB13-Pad26) -> /MODE_VA
- U1 pad 27: unconnected-(U1-PB14-Pad27) -> /MODE_PTT
- U1 pad 28: unconnected-(U1-PB15-Pad28) -> /MODE_M
- U1 pad 29: unconnected-(U1-PA8-Pad29) -> /PTT_IN
- U1 pad 30: unconnected-(U1-PA9-Pad30) -> /PTT_OUT
- U1 pad 32: unconnected-(U1-PA11-Pad32) -> /USB_D-
- U1 pad 33: unconnected-(U1-PA12-Pad33) -> /USB_D+
Routing:
- net /USB_D-: track 0.00 -> 43.4 mm, vias 0 -> 1
- net /USB_D+: track 0.00 -> 42.5 mm, vias 0 -> 1
- net Net-(U3-IN+): track 0.00 -> 21.2 mm
- net VBUS: track 0.00 -> 20.1 mm
- net Net-(U3-IN-): track 0.00 -> 19.9 mm
- net GND: track 0.00 -> 13.7 mm, vias 0 -> 9
- net /SWCLK: track 0.00 -> 10.8 mm
- net /SWDIO: track 0.00 -> 9.53 mm
- net Net-(J4-Pin_1): track 0.00 -> 7.39 mm
- net Net-(J2-CC2): track 0.00 -> 5.64 mm
- net Net-(J4-Pin_2): track 0.00 -> 3.56 mm
- net +3V3: track 0.00 -> 3.22 mm, vias 0 -> 2
- net /IN-: track 0.00 -> 1.98 mm
- net /IN+: track 0.00 -> 1.98 mm
- net Net-(J2-CC1): track 0.00 -> 1.90 mm
- added copper zone on In2.Cu, net +3V3
- added copper zone on In1.Cu, net GND
Other:
- board outline added: 40 x 80 mm
- copper layers 2 -> 4

Commit message: pcb routing
Parts:
- added H1: MountingHole_Pad, MountingHole:MountingHole_2.7mm_M2.5_ISO7380_Pad, F.Cu at (131.5, 142.0)
- added H2: MountingHole_Pad, MountingHole:MountingHole_2.7mm_M2.5_ISO7380_Pad, F.Cu at (165.5, 142.0)
- added H3: MountingHole_Pad, MountingHole:MountingHole_2.7mm_M2.5_ISO7380_Pad, F.Cu at (131.5, 68.0)
- moved C10 79.7 mm to (165.8, 135.7), turned to -90 degrees
- moved R4 76.5 mm to (166.0, 124.2), turned to -90 degrees
- moved C11 74.4 mm to (165.0, 128.2)
- moved R7 70.6 mm to (157.3, 133.0), turned to 180 degrees
- moved R6 68.5 mm to (157.3, 127.2)
- moved C9 64.4 mm to (159.5, 101.5), turned to -90 degrees
- moved C14 64.2 mm to (148.6, 115.8)
- moved C1 63.4 mm to (149.2, 107.9), turned to 90 degrees
- moved C5 62.7 mm to (155.1, 104.2)
- moved C4 62.5 mm to (152.9, 106.8)
- moved C12 61.7 mm to (153.0, 126.8), turned to 180 degrees
- moved C20 61.0 mm to (156.2, 97.8)
- moved C8 59.8 mm to (155.4, 102.5)
- moved C7 59.6 mm to (154.5, 99.5)
- moved C17 59.3 mm to (159.2, 73.8)
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Connections:
- U1 pad 17: unconnected-(U1-PA7-Pad17) -> /SD
Routing:
- net /VHI: track 0.00 -> 63.7 mm, vias 0 -> 2
- net /EN: track 0.00 -> 58.7 mm, vias 0 -> 2
- net /PTT_OUT: track 0.00 -> 50.3 mm, vias 0 -> 2
- net /PTT_IN: track 0.00 -> 49.8 mm, vias 0 -> 2
- net /MODE_M: track 0.00 -> 45.4 mm, vias 0 -> 2
- net /MODE_PTT: track 0.00 -> 44.3 mm, vias 0 -> 2
- net /MODE_VA: track 0.00 -> 43.3 mm, vias 0 -> 2
- net /MODE_C: track 0.00 -> 43.1 mm, vias 0 -> 2
- net /BUSY: track 0.00 -> 40.9 mm, vias 0 -> 2
- net GND: track 13.7 -> 53.2 mm, vias 9 -> 44
- net /DIO1: track 0.00 -> 29.2 mm, vias 0 -> 2
- net +3V3: track 3.22 -> 26.9 mm, vias 2 -> 10
- net /SW: track 0.00 -> 22.7 mm
- net /MISO: track 0.00 -> 21.5 mm
- net /MOSI: track 0.00 -> 20.1 mm
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- added copper zone on F.Cu, net /VHI
- added copper zone on F.Cu, net GND
- added copper zone on F.Cu, net VBUS
- added copper zone on F.Cu, net VDDA

Commit message: silkscreen, 3d models
Parts:
- J3: moved to B.Cu
- moved J3 4.01 mm to (155.5, 121.5), turned to 0 degrees
Routing:
- net Net-(MK1-+): track 6.70 -> 9.90 mm
Other:
- board text added: "+"
- board text added: "-"
- board text added: "868 MHz"
- board text added: "868 MHz LoRa walkie-talkie"
- board text added: "BAT"
- board text added: "Copyright © 2026"
- board text added: "OUT"
- board text added: "Olivér Pirger"
- board text added: "PTT"
- board text added: "PWR"
- board text added: "SEL"
- board text added: "SWD"
- board text added: "mini-talkie"

Commit message: continue 3d model
Connections:
- J4 pad 1: Net-(J4-Pin_1) -> /O-
- J4 pad 2: Net-(J4-Pin_2) -> /O+
- U3 pad 5: Net-(J4-Pin_1) -> /O+
- U3 pad 8: Net-(J4-Pin_2) -> /O-
Routing:
- net /O-: track 0.00 -> 14.6 mm
- net Net-(J4-Pin_2): track 12.3 -> 0.00 mm
- net Net-(J4-Pin_1): track 8.65 -> 0.00 mm
- net /O+: track 0.00 -> 7.23 mm
Changed lines of the file:
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@@
 			(remove_unused_layers no)
 			(roundrect_rratio 0.208333)
-			(net "Net-(J4-Pin_1)")
+			(net "/O-")
 			(pinfunction "Pin_1_1")
 			(pintype "passive")
@@
 			(layers "*.Cu" "*.Mask")
 			(remove_unused_layers no)
-			(net "Net-(J4-Pin_2)")
+			(net "/O+")
 			(pinfunction "Pin_2_2")
 			(pintype "passive")
@@
 			)
 		)
-		(property "MPN" ""
+		(property "MPN" "OS102011MA1QN1"
 			(at 0 0 270)
 			(unlocked yes)
@@
 			)
 		)
-		(property "MPN" ""
+		(property "MPN" "114993390"
 			(at 0 0 90)
 			(unlocked yes)
@@
 			)
 		)
-		(property "MPN" ""
+		(property "MPN" "MCP73831T-2ACI/OT"
 			(at 0 0 270)
 			(unlocked yes)
@@
 			)
 		)
-		(property "MPN" ""
+		(property "MPN" "TOW-3050P-B-R "
 			(at 0 0 180)
 			(unlocked yes)
@@
 			)
 		)
-		(property "MPN" ""
+		(property "MPN" "PAM8302AASCR"
 			(at 0 0 90)
 			(unlocked yes)
@@
 			(layers "F.Cu" "F.Mask" "F.Paste")
 			(roundrect_rratio 0.25)
-			(net "Net-(J4-Pin_1)")
+			(net "/O+")
 			(pinfunction "OUT+_5")
 			(pintype "output")
@@
 			(layers "F.Cu" "F.Mask" "F.Paste")
 			(roundrect_rratio 0.25)
-			(net "Net-(J4-Pin_2)")
+			(net "/O-")
 			(pinfunction "OUT-_8")
 			(pintype "output")
@@
 			)
 		)
-		(property "MPN" ""
+		(property "MPN" "RT9080-33GJ5"
 			(at 0 0 90)
 			(unlocked yes)
@@
 			)
 		)
+		(attr exclude_from_bom)
 		(duplicate_pad_numbers_are_jumpers no)
 		(fp_circle
@@
 			)
 		)
-		(property "MPN" ""
+		(property "MPN" "B3F-3152"
 			(at 0 0 270)
 			(unlocked yes)
@@
 			)
 		)
-		(property "MPN" ""
+		(property "MPN" "OS103011MA7QP1C"
 			(at 0 0 90)
 			(unlocked yes)
@@
 			)
 		)
-		(property "MPN" ""
+		(property "MPN" "STM32H503CBT6"
 			(at 0 0 180)
 			(unlocked yes)
@@
 			)
 		)
+		(attr exclude_from_bom)
 		(duplicate_pad_numbers_are_jumpers no)
 		(fp_circle
@@
 	)
 	(segment
-		(start 160.3625 77.8875)
-		(end 165.5 72.75)
-		(width 0.4)
-		(layer "F.Cu")
-		(net "Net-(J4-Pin_1)")
-	)
-	(segment
-		(start 158.975 77.8875)
-		(end 160.3625 77.8875)
-		(width 0.4)
-		(layer "F.Cu")
-		(net "Net-(J4-Pin_1)")
-	)
-	(segment
-		(start 162.55 71.8)
-		(end 163.5 72.75)
-		(width 0.4)
-		(layer "F.Cu")
-		(net "Net-(J4-Pin_2)")
-	)
-	(segment
-		(start 158.829358 71.8)
-		(end 162.55 71.8)
-		(width 0.4)
-		(layer "F.Cu")
-		(net "Net-(J4-Pin_2)")
-	)
-	(segment
-		(start 156.55 74.079358)
-		(end 158.829358 71.8)
-		(width 0.4)
-		(layer "F.Cu")
-		(net "Net-(J4-Pin_2)")
-	)
-	(segment
-		(start 157.025 77.8875)
-		(end 156.55 77.4125)
-		(width 0.4)
-		(layer "F.Cu")
-		(net "Net-(J4-Pin_2)")
-	)
-	(segment
-		(start 156.55 77.4125)
-		(end 156.55 74.079358)
-		(width 0.4)
-		(layer "F.Cu")
-		(net "Net-(J4-Pin_2)")
-	)
-	(segment
 		(start 160.05 75.5)
 		(end 160.75 75.5)
@@
 	)
 	(segment
+		(start 156.25 127.425)
+		(end 156.425 127.25)
+		(width 0.2)
+		(layer "F.Cu")
+		(net "Net-(U4-STAT)")
+	)
+	(segment
+		(start 156.25 128.975)
+		(end 156.25 127.425)
+		(width 0.2)
+		(layer "F.Cu")
+		(net "Net-(U4-STAT)")
+	)
+	(segment
 		(start 154.075 124.675)
 		(end 157.5 121.25)
@@
 	)
 	(segment
-		(start 156.25 127.425)
-		(end 156.425 127.25)
-		(width 0.2)
-		(layer "F.Cu")
-		(net "Net-(U4-STAT)")
-	)
-	(segment
-		(start 156.25 128.975)
-		(end 156.25 127.425)
-		(width 0.2)
-		(layer "F.Cu")
-		(net "Net-(U4-STAT)")
-	)
-	(segment
 		(start 157.425 135.825)
 		(end 157.75 135.5)
@@
 		(net "/SWCLK")
 	)
+	(segment
+		(start 157.025 77.8875)
+		(end 156.55 77.4125)
+		(width 0.4)
+		(layer "F.Cu")
+		(net "/O-")
+	)
+	(segment
+		(start 156.55 77.4125)
+		(end 156.55 74.079358)
+		(width 0.4)
+		(layer "F.Cu")
+		(net "/O-")
+	)
+	(segment
+		(start 164.225 71.475)
+		(end 165.5 72.75)
+		(width 0.4)
+		(layer "F.Cu")
+		(net "/O-")
+	)
+	(segment
+		(start 156.55 74.079358)
+		(end 159.154358 71.475)
+		(width 0.4)
+		(layer "F.Cu")
+		(net "/O-")
+	)
+	(segment
+		(start 159.154358 71.475)
+		(end 164.225 71.475)
+		(width 0.4)
+		(layer "F.Cu")
+		(net "/O-")
+	)
+	(segment
+		(start 158.975 77.8875)
+		(end 159.35245 77.8875)
+		(width 0.4)
+		(layer "F.Cu")
+		(net "/O+")
+	)
+	(segment
+		(start 159.35245 77.8875)
+		(end 163.5 73.73995)
+		(width 0.4)
+		(layer "F.Cu")
+		(net "/O+")
+	)
+	(segment
+		(start 163.5 73.73995)
+		(end 163.5 72.75)
+		(width 0.4)
+		(layer "F.Cu")
+		(net "/O+")
+	)
 	(zone
