File: pcb/mini-talkie.kicad_sch (KiCad schematic)
At the start: 3 parts, among them U1 STM32H503CBTx, U2 Wio-SX1262

Commit message: switches, power supply
Parts:
- added C1, C2: 2.2u, symbol Device:C
- added C10, C11: 10u, symbol Device:C
- added C3, C4, C5, C6, C7, C9: 100n, symbol Device:C
- added C8: 4.7u, symbol Device:C
- added D1: PMEG3020EH, Diode_SMD:D_SMA_Handsoldering, symbol Diode:PMEG3020EH
- added J1: SWD, Connector_JST:JST_SH_BM03B-SRSS-TB_1x03-1MP_P1.00mm_Vertical, symbol Connector_Generic_MountingPin:Conn_01x03_MountingPin
- added J2: USB_C_Receptacle_USB2.0_16P, Connector_USB:USB_C_Receptacle_GCT_USB4085, symbol Connector:USB_C_Receptacle_USB2.0_16P
- added Q1: AO3401A, Package_TO_SOT_SMD:SOT-23, symbol Transistor_FET:AO3401A
- added R1, R4, R5: 10k, symbol Device:R
- added R2, R3: 5.1k, symbol Device:R
- added SW1: SW_SP3T, Mini_Talkie:CK_SW_SP3T_OS103011MA7QP1C, symbol Switch:SW_SP3T
- added SW2: SW_SPDT, Button_Switch_THT:SW_Slide_SPDT_Angled_CK_OS102011MA1Q, symbol Switch:SW_SPDT
- added SW3: SW_SPST, Button_Switch_THT:SW_SPST_Omron_B3F-315x_Angled, symbol Switch:SW_SPST
- added TP1: ~{RST}, TestPoint:TestPoint_Pad_D2.0mm, symbol Connector:TestPoint
- added TP2: BOOT0, symbol Connector:TestPoint
- added U3: PAM8302AAS, Package_SO:MSOP-8_3x3mm_P0.65mm, symbol Amplifier_Audio:PAM8302AAS
- added U4: MCP73831-2-OT, Package_TO_SOT_SMD:SOT-23-5, symbol Battery_Management:MCP73831-2-OT
- added U5: RT9080, Package_TO_SOT_SMD:TSOT-23-5, symbol mini-talkie:RT9080
Connections:
- net GND: now also U1.23 (VSS), U1.35 (VSS), U1.47 (VSS), U1.8 (VSSA), C1.1, C10.2, C11.2, C2.1, C3.2, C4.2, C5.2, C6.2, C7.2, C8.2, C9.2, J1.2 (Pin_2), J1.MP (MountPin), J2.A1 (GND), J2.A12 (GND), J2.B1 (GND), J2.B12 (GND), J2.SH (SHIELD), R1.1, R2.2, R3.2, R5.2, U5.2 (GND), U5.4 (GND)
- net +3V3: now reaches U1.1 (VBAT)
- net +3V3: now also U1.24 (VDD), U1.36 (VDD), U1.48 (VDD), U1.9 (VDDA), C11.1, C3.1, C4.1, C5.1, C6.1, C7.1, C8.1, U5.5 (VOUT)
- net at U1.22 (VCAP): now also C2.2
- net SWDIO: now reaches U1.34 (PA13(JTMS)
- net SWDIO: now also J1.3 (Pin_3)
- net SWCLK: now reaches U1.37 (PA14(JTCK)
- net SWCLK: now also J1.1 (Pin_1)
- net at U1.44 (BOOT0): now also R1.2, TP2.1
- net at U1.46 (VCAP): now also C1.2
- net at U1.7 (NRST): now also C9.1, TP1.1
- new net: J2.A5 (CC1), R3.1
- new net: J2.B5 (CC2), R2.1
- new net: C10.1, D1.1 (K), Q1.2 (S), R4.1, U5.1 (VIN)
- new net: R4.2, U5.3 (EN)
- new net +BATT: Q1.3 (D)
- new net USB_D+: J2.A6 (D+), J2.B6 (D+)
- new net USB_D-: J2.A7 (D-), J2.B7 (D-)
- new net VBUS: D1.2 (A), J2.A4 (VBUS), J2.A9 (VBUS), J2.B4 (VBUS), J2.B9 (VBUS), Q1.1 (G), R5.1
- no-connect marks 0 -> 4
Other:
- moved on the sheet: MK1, U1, U2

Commit message: schematic almost done
Parts:
- added C12, C13, C20: 10u, Capacitor_SMD:C_0805_2012Metric_Pad1.18x1.45mm_HandSolder, symbol Device:C
- added C14, C18, C19: 100n, Capacitor_SMD:C_0603_1608Metric_Pad1.08x0.95mm_HandSolder, symbol Device:C
- added C15, C16: 1u, Capacitor_SMD:C_0603_1608Metric_Pad1.08x0.95mm_HandSolder, symbol Device:C
- added C17: 10u, Capacitor_SMD:C_0603_1608Metric_Pad1.08x0.95mm_HandSolder, symbol Device:C
- added D2: ORANGE, LED_SMD:LED_0805_2012Metric_Pad1.15x1.40mm_HandSolder, symbol Device:LED
- added FB1: 600@100, Inductor_SMD:L_0603_1608Metric_Pad1.05x0.95mm_HandSolder, symbol Device:FerriteBead
- added J3: BATT, Connector_JST:JST_PH_S2B-PH-K_1x02_P2.00mm_Horizontal, symbol Connector_Generic:Conn_01x02
- added J4: SPEAKER, Connector_JST:JST_PH_S2B-PH-K_1x02_P2.00mm_Horizontal, symbol Connector_Generic:Conn_01x02
- added R6: 10k, Resistor_SMD:R_0603_1608Metric_Pad0.98x0.95mm_HandSolder, symbol Device:R
- added R7: 5.1k, Resistor_SMD:R_0603_1608Metric_Pad0.98x0.95mm_HandSolder, symbol Device:R
- added R8: 1k, Resistor_SMD:R_0805_2012Metric_Pad1.20x1.40mm_HandSolder, symbol Device:R
- C1, C2, C3, C4, C5, C6, C7, C9: footprint (none) -> Capacitor_SMD:C_0603_1608Metric_Pad1.08x0.95mm_HandSolder
- C10, C11: footprint (none) -> Capacitor_SMD:C_0805_2012Metric_Pad1.18x1.45mm_HandSolder
- C8: value 4.7u -> 10u; footprint (none) -> Capacitor_SMD:C_0805_2012Metric_Pad1.18x1.45mm_HandSolder
- R1, R2, R3, R4, R5: footprint (none) -> Resistor_SMD:R_0603_1608Metric_Pad0.98x0.95mm_HandSolder
- TP2: footprint (none) -> TestPoint:TestPoint_Pad_D2.0mm
Connections:
- net +3V3: now also U2.8 (VCC), U3.6 (VDD), C13.1, C14.1, C16.1, C17.1, FB1.2, R8.1; no longer C7.1, U1.9 (VDDA)
- net +BATT: now also U4.3 (V_{BAT}), C12.1, J3.2 (Pin_2)
- net GND: now also MK1.1 (-), SW2.1 (A), U3.7 (GND), U4.2 (V_{SS}), C12.2, C13.2, C14.2, C16.2, C17.2, C20.2, J3.1 (Pin_1), R7.1
- net VBUS: now also U4.4 (V_{DD}), D2.2 (A)
- net SW: now reaches U2.1 (RF_SW)
- net SW: now also U1.38 (PA15(JTDI))
- net BUSY: now reaches U2.11 (BUSY)
- net BUSY: now also U1.2 (PC13)
- net DIO1: now reaches U2.12 (DIO1)
- net DIO1: now also U1.43 (PB7)
- net MISO: now reaches U2.2 (MISO)
- net MISO: now also U1.40 (PB4(NJTRST))
- net MOSI: now reaches U2.3 (MOSI)
- net MOSI: now also U1.41 (PB5)
- net SCK: now reaches U2.4 (SCK)
- net SCK: now also U1.39 (PB3(JTDO)
- net RST: now reaches U2.5 (~{RST})
- net RST: now also U1.42 (PB6)
- net NSS: now reaches U2.6 (NSS)
- net NSS: now also U1.45 (PB8)
- net SD: now reaches U3.1 (~{SD})
- net at U3.3 (IN+): now also C18.2
- net at U3.4 (IN-): now also C19.2
- net at U3.5 (OUT+): now also J4.1 (Pin_1)
- net at U3.8 (OUT-): now also J4.2 (Pin_2)
- net at U4.1 (STAT): now also R6.1
- net at U4.5 (PROG): now also R7.2
- net VHI: now reaches C10.1, D1.1 (K), Q1.2 (S), U5.1 (VIN)
- net VHI: now also SW2.3 (C); no longer R4.1
- net at MK1.2 (+): now also C15.2, R8.2
- net EN: now reaches SW2.2 (B)
- net EN: now also R4.1
- net IN+: now reaches U1.14 (PA4)
- net IN+: now also C18.1
- net IN-: now reaches U1.15 (PA5)
- net IN-: now also C19.1
- net MIC: now reaches U1.18 (PB0)
- net MIC: now also C15.1
- new net: D2.1 (K), R6.2
- new net VDDA: C20.1, C7.1, FB1.1, U1.9 (VDDA)
- no-connect marks 4 -> 5
Other:
- moved on the sheet: C3, C4, C5, C6, C7, C8, J1, MK1, SW1, SW2, SW3, U2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

Commit message: get started with layout
Connections:
- net USB_D+: now also U1.33 (PA12)
- net USB_D-: now also U1.32 (PA11)
- net MODE_VA: now reaches SW1.1
- net MODE_VA: now also U1.26 (PB13)
- net MODE_PTT: now reaches SW1.2
- net MODE_PTT: now also U1.27 (PB14)
- net MODE_C: now reaches SW1.3
- net MODE_C: now also U1.25 (PB12)
- net MODE_M: now reaches SW1.4
- net MODE_M: now also U1.28 (PB15)
- net PTT_IN: now reaches SW3.1 (A)
- net PTT_IN: now also U1.29 (PA8)
- net PTT_OUT: now reaches SW3.2 (B)
- net PTT_OUT: now also U1.30 (PA9)
Other:
- moved on the sheet: SW1, SW3

Commit message: pcb routing
Parts:
- added H1, H2, H3: MountingHole_Pad, MountingHole:MountingHole_2.7mm_M2.5_ISO7380_Pad, symbol Mechanical:MountingHole_Pad
Connections:
- net GND: now also H1.1, H2.1, H3.1
- net SD: now also U1.17 (PA7)
- no-connect marks 5 -> 16
Other:
- moved on the sheet: C13, C14, SW1, SW3, U2

Commit message: start bom
Parts:
- MK1: MPN (none) -> TOW-3050P-B-R
- SW1: MPN (none) -> OS103011MA7QP1C
- SW2: MPN (none) -> OS102011MA1QN1
- SW3: MPN (none) -> B3F-3152
- TP1, TP2: now left out of the parts list
- U1: MPN (none) -> STM32H503CBT6
- U2: MPN (none) -> 114993390
- U3: MPN (none) -> PAM8302AASCR
- U4: MPN (none) -> MCP73831T-2ACI/OT
- U5: MPN (none) -> RT9080-33GJ5

Commit message: continue 3d model
Connections:
- net O+: now reaches U3.5 (OUT+)
- net O+: now also J4.2 (Pin_2); no longer J4.1 (Pin_1)
- net O-: now reaches U3.8 (OUT-)
- net O-: now also J4.1 (Pin_1); no longer J4.2 (Pin_2)
Other:
- moved on the sheet: J4

Commit message: continue bom
Parts:
- D1: value PMEG3020EH -> B0520WS-7-F
